Commit message: Update navigation stack - Add display.launch to launch RViz using the URDF - Update the chassis.urdf to include temporary geometry - Correction in gmu_rtx_ground.urdf robot tag

File: ROS/losi_launch/urdf/chassis.urdf.xacro (robot description, xacro)
@@ -5,8 +5,9 @@
             <visual>
                 <origin rpy="0 0 0" xyz="-0.2 0 -0.12"/>
-                <!-- <geometry> -->
+                <geometry>
                     <!-- <mesh filename="file:///home/aniket/Documents/MPPI_vertiFormer/mesh/v4w.obj" scale="1 1 1"/> -->
                     <!-- <mesh filename="package://losi_launch/meshes/v4w.obj" scale="1 1 1"/> -->
-                <!-- </geometry> -->
+                    <box size="1.0 1.3 1.1"/>
+                </geometry>
                 <material name="grey"/>
             </visual>
@@ -18,8 +19,9 @@
             <collision>
               <origin rpy="1.5708 0 0" xyz="-0.2 0 -0.1"/>
-                <!-- <geometry> -->
+                <geometry>
                     <!-- <mesh filename="file:///home/aniket/Documents/MPPI_vertiFormer/mesh/v4w.stl" scale="1 1 1"/> -->
                     <!-- <mesh filename="package://losi_launch/meshes/v4w.stl" scale="1 1 1"/> -->
-                <!-- </geometry> -->
+                    <box size="1.0 1.3 1.1"/>
+                </geometry>
             </collision>
         </link>

File: ROS/losi_launch/urdf/gmu_rtx_ground.urdf.xacro (robot description, xacro)
@@ -1,5 +1,5 @@
 <?xml version="1.0"?>
 <!-- Top-Level URDF for Ground Robot -->
-<xacro:robot name="gmu-rtx-ground" xmlns:xacro="http://ros.org/wiki/xacros">
+<robot name="gmu-rtx-ground" xmlns:xacro="http://ros.org/wiki/xacros">
   <!-- Load chassis -->
   <xacro:include filename="chassis.urdf.xacro"/>
@@ -11,3 +11,3 @@
   <xacro:chassis/>
   <xacro:sensors/>
-</xacro:robot>
+</robot>

Commit message: Update chassis.urdf - Zero out origin - Minor tweaks to shape geomtry - Ensure wheels rotated on correct axis wrt base_link - Correctly model front axle - Model steering servo - Model transmission servo

File: ROS/losi_launch/urdf/chassis.urdf.xacro (robot description, xacro)
@@ -4,9 +4,9 @@
         <link name="base_link">
             <visual>
-                <origin rpy="0 0 0" xyz="-0.2 0 -0.12"/>
+                <origin rpy="0 0 0" xyz="0 0 0"/>
                 <geometry>
                     <!-- <mesh filename="file:///home/aniket/Documents/MPPI_vertiFormer/mesh/v4w.obj" scale="1 1 1"/> -->
                     <!-- <mesh filename="package://losi_launch/meshes/v4w.obj" scale="1 1 1"/> -->
-                    <box size="1.0 1.3 1.1"/>
+                    <box size="0.6 0.3 0.1"/>
                 </geometry>
                 <material name="grey"/>
@@ -18,100 +18,134 @@
             </intertial>
             <collision>
-              <origin rpy="1.5708 0 0" xyz="-0.2 0 -0.1"/>
+              <origin rpy="0 0 0" xyz="0 0 0"/>
                 <geometry>
                     <!-- <mesh filename="file:///home/aniket/Documents/MPPI_vertiFormer/mesh/v4w.stl" scale="1 1 1"/> -->
                     <!-- <mesh filename="package://losi_launch/meshes/v4w.stl" scale="1 1 1"/> -->
-                    <box size="1.0 1.3 1.1"/>
+                    <box size="0.6 0.3 0.1"/>
                 </geometry>
             </collision>
         </link>
-        <!-- Front axle -->
-        <joint name="front_left_steering_joint" type="revolute">
+        <!-- Steering servo -->
+        <link name="steering_servo_link">
+            <visual>
+                <origin xyz="0.3 0 0.05" rpy="0 0 0"/>
+                <geometry>
+                    <box size="0.05 0.05 0.05"/>
+                </geometry>
+                <material name="blue"/>
+            </visual>
+        </link>
+        <joint name="steering_servo_joint" type="fixed">
             <parent link="base_link"/>
-            <child link="front_left_wheel_link"/>
-            <origin xyz="0.3 0.18 -0.07" rpy="0 0 0"/>
-            <axis xyz="0 0 1"/> <!-- steer around Z (yaw) -->
-            <limit lower="-0.5236" upper="0.5236" effort="10" velocity="1.0"/>
+                <child link="steering_servo_link"/>
+            <origin xyz="0.3 0 0.05" rpy="0 0 0"/>
         </joint>
+        <!-- Transmission servo -->
+        <link name="transmission_servo_link">
+            <visual>
+                <origin xyz="-0.2 0 0.05" rpy="0 0 0"/>
+                <geometry>
+                    <box size="0.05 0.05 0.05"/>
+                </geometry>
+                <material name="blue"/>
+            </visual>
+        </link>
+        <joint name="transmission_servo_joint" type="fixed">
+            <parent link="base_link"/>
+                <child link="transmission_servo_link"/>
+            <origin xyz="-0.2 0 0.05" rpy="0 0 0"/>
+        </joint>
+        <!-- Front steering axle -->
+        <link name="front_axle_link">
+            <visual>
+                <origin xyz="0.25 0 0" rpy="0 0 0"/>
+                <geometry>
+                    <box size="0.1 0.6 0.05"/>
+                </geometry>
+                <material name="red"/>
+            </visual>
+        </link>
+        <joint name="steering_joint" type="revolute">
+            <parent link="base_link"/>
+            <child link="front_axle_link"/>
+            <origin xyz="0.25 0 0" rpy="0 0 0"/>
+            <axis xyz="0 0 1"/>
+            <limit lower="-0.5236" upper="0.5236" effort="5" velocity="1.0"/>
+        </joint>
+        <!-- Front left wheel -->
         <link name="front_left_wheel_link">
             <visual>
-                <origin xyz="0 0 0" rpy="0 0 0"/>
-                <geometry>
-                    <cylinder radius="0.07" length="0.04"/>
-                </geometry>
-                <material name="grey"/>
+            <origin xyz="0 0.2 0" rpy="1.5708 0 0"/>
+            <geometry>
+                <cylinder radius="0.07" length="0.04"/>
+            </geometry>
+            <material name="black"/>
             </visual>
-            <inertial>
-                <origin xyz="0 0 0" rpy="0 0 0"/>
-                <mass value="0.5"/>
-                <inertia ixx="1e-3" iyy="1e-3" izz="1e-3"
-                        ixy="0" ixz="0" iyz="0"/>
-            </inertial>
         </link>
-        <joint name="front_right_steering_joint" type="revolute">
-            <parent link="base_link"/>
-            <child link="front_right_wheel_link"/>
-            <origin xyz="0.3 -0.18 -0.07" rpy="0 0 0"/>
-            <axis xyz="0 0 1"/>
-            <limit lower="-0.5236" upper="0.5236" effort="10" velocity="1.0"/>
+        <joint name="front_left_wheel_joint" type="fixed">
+            <parent link="front_axle_link"/>
+            <child link="front_left_wheel_link"/>
+            <origin xyz="0 0.2 0" rpy="0 0 0"/>
         </joint>
+        <!-- Front right wheel -->
         <link name="front_right_wheel_link">
             <visual>
-                <origin xyz="0 0 0" rpy="0 0 0"/>
-                <geometry>
-                    <cylinder radius="0.07" length="0.04"/>
-                </geometry>
-                <material name="grey"/>
+            <origin xyz="0 -0.2 0" rpy="1.5708 0 0"/>
+            <geometry>
+                <cylinder radius="0.07" length="0.04"/>
+            </geometry>
+            <material name="black"/>
             </visual>
-            <inertial>
-                <origin xyz="0 0 0" rpy="0 0 0"/>
-                <mass value="0.5"/>
-                <inertia ixx="1e-3" iyy="1e-3" izz="1e-3"
-                        ixy="0" ixz="0" iyz="0"/>
-            </inertial>
         </link>
-        <!-- Back axle -->
-        <joint name="rear_left_wheel_joint" type="continuous">
+        <joint name="front_right_wheel_joint" type="fixed">
+            <parent link="front_axle_link"/>
+            <child link="front_right_wheel_link"/>
+            <origin xyz="0 -0.2 0" rpy="0 0 0"/>
+        </joint>
+        <!-- Rear axle -->
+        <link name="rear_axle_link">
+            <visual>
+            <origin xyz="-0.25 0 0" rpy="0 0 0"/>
+            <geometry>
+                <box size="0.1 0.6 0.05"/>
+            </geometry>
+            <material name="red"/>
+            </visual>
+        </link>
+        <joint name="rear_axle_joint" type="fixed">
             <parent link="base_link"/>
-            <child link="rear_left_wheel_link"/>
-            <origin xyz="-0.3 0.18 -0.07" rpy="0 0 0"/>
-            <axis xyz="0 1 0"/>
+            <child link="rear_axle_link"/>
+            <origin xyz="-0.25 0 0" rpy="0 0 0"/>
         </joint>
+        <!-- Rear left wheel -->
         <link name="rear_left_wheel_link">
             <visual>
-                <origin xyz="0 0 0" rpy="0 0 0"/>
-                <geometry>
-                    <cylinder radius="0.07" length="0.04"/>
-                </geometry>
-                <material name="grey"/>
+            <origin xyz="0 0.2 0" rpy="1.5708 0 0"/>
+            <geometry>
+                <cylinder radius="0.07" length="0.04"/>
+            </geometry>
+            <material name="black"/>
             </visual>
-            <inertial>
-                <origin xyz="0 0 0" rpy="0 0 0"/>
-                <mass value="0.5"/>
-                <inertia ixx="1e-3" iyy="1e-3" izz="1e-3"
-                        ixy="0" ixz="0" iyz="0"/>
-            </inertial>
         </link>
-        <joint name="rear_right_wheel_joint" type="continuous">
-            <parent link="base_link"/>
-            <child link="rear_right_wheel_link"/>
-            <origin xyz="-0.3 -0.18 -0.07" rpy="0 0 0"/>
-            <axis xyz="0 1 0"/>
+        <joint name="rear_left_wheel_joint" type="fixed">
+            <parent link="rear_axle_link"/>
+            <child link="rear_left_wheel_link"/>
+            <origin xyz="0 0.2 0" rpy="0 0 0"/>
         </joint>
+        <!-- Rear right wheel -->
         <link name="rear_right_wheel_link">
             <visual>
-                <origin xyz="0 0 0" rpy="0 0 0"/>
-                <geometry>
-                    <cylinder radius="0.07" length="0.04"/>
-                </geometry>
-                <material name="grey"/>
+            <origin xyz="0 -0.2 0" rpy="1.5708 0 0"/>
+            <geometry>
+                <cylinder radius="0.07" length="0.04"/>
+            </geometry>
+            <material name="black"/>
             </visual>
-            <inertial>
-                <origin xyz="0 0 0" rpy="0 0 0"/>
-                <mass value="0.5"/>
-                <inertia ixx="1e-3" iyy="1e-3" izz="1e-3"
-                        ixy="0" ixz="0" iyz="0"/>
-            </inertial>
         </link>
+        <joint name="rear_right_wheel_joint" type="fixed">
+            <parent link="rear_axle_link"/>
+            <child link="rear_right_wheel_link"/>
+            <origin xyz="0 -0.2 0" rpy="0 0 0"/>
+        </joint>
     </xacro:macro>
 </robot>

File: ROS/losi_launch/urdf/materials.xacro (robot description, xacro)
@@ -10,3 +10,9 @@
         <color rgba="0.5 0.5 0.5 1"/>
     </material>
+    <material name="black">
+        <color rgba="0 0 0 1"/>
+    </material>
+    <material name="red">
+        <color rgba="1 0.5 0.2 0.4"/>
+    </material>
 </robot>

Commit message: Increase model tire radius

File: ROS/losi_launch/urdf/chassis.urdf.xacro (robot description, xacro)
@@ -78,5 +78,5 @@
             <origin xyz="0 0.2 0" rpy="1.5708 0 0"/>
             <geometry>
-                <cylinder radius="0.07" length="0.04"/>
+                <cylinder radius="0.12" length="0.04"/>
             </geometry>
             <material name="black"/>
@@ -93,5 +93,5 @@
             <origin xyz="0 -0.2 0" rpy="1.5708 0 0"/>
             <geometry>
-                <cylinder radius="0.07" length="0.04"/>
+                <cylinder radius="0.12" length="0.04"/>
             </geometry>
             <material name="black"/>
@@ -123,5 +123,5 @@
             <origin xyz="0 0.2 0" rpy="1.5708 0 0"/>
             <geometry>
-                <cylinder radius="0.07" length="0.04"/>
+                <cylinder radius="0.12" length="0.04"/>
             </geometry>
             <material name="black"/>
@@ -138,5 +138,5 @@
             <origin xyz="0 -0.2 0" rpy="1.5708 0 0"/>
             <geometry>
-                <cylinder radius="0.07" length="0.04"/>
+                <cylinder radius="0.12" length="0.04"/>
             </geometry>
             <material name="black"/>

Commit message: Updates to symlinks and ekf and losi config/launch files

File: ROS/losi_launch/urdf/chassis.urdf.xacro (robot description, xacro)
@@ -66,5 +66,6 @@
             </visual>
         </link>
-        <joint name="steering_joint" type="revolute">
+        <!-- change back to type=revolute and publish steering joint state for steering sim -->
+        <joint name="steering_joint" type="fixed">
             <parent link="base_link"/>
             <child link="front_axle_link"/>
