Commit message: Add LiDAR module to URDF

File: ROS/losi_launch/urdf/sensors.urdf.xacro (robot description, xacro)
@@ -42,4 +42,24 @@
         <origin xyz="0 0 0.15" rpy="0 0 0"/>
     </joint>
+    <!-- LiDAR link -->
+    <link name="lidar_link">
+        <visual>
+            <origin xyz="0 0 0" rpy="0 0 0"/>
+            <geometry>
+                <box size="0.02 0.02 0.02"/>
+            </geometry>
+            <material name="black"/>
+        </visual>
+        <inertial>
+            <origin xyz="0 0 0" rpy="0 0 0"/>
+            <mass value="0.001"/>
+            <inertia ixx="1e-6" ixy="0" ixz="0" iyy="1e-6" iyz="0" izz="1e-6"/>
+        </inertial>
+    </link>
+    <joint name="lidar_joint" type="fixed">
+        <parent link="base_link"/>
+        <child link="lidar_link"/>
+        <origin xyz="0 0 0.2" rpy="0 0 0"/>
+    </joint>
   </xacro:macro>
 </robot>

Commit message: Refactored ROS

File: ROS/losi_launch/urdf/sensors.urdf.xacro (robot description, xacro)
@@ -23,5 +23,5 @@
     </joint>
     <!-- GPS link -->
-    <link name="gps_link">
+    <link name="rover">
         <visual>
             <origin xyz="0 0 0" rpy="0 0 0"/>
@@ -39,5 +39,5 @@
     <joint name="gps_joint" type="fixed">
         <parent link="base_link"/>
-        <child link="gps_link"/>
+        <child link="rover"/>
         <origin xyz="0 0 0.15" rpy="0 0 0"/>
     </joint>
